Commit message: created gazebo pkg

File: widowx_arm_description/urdf/widowx.urdf.xacro (robot description, xacro)
@@ -1,6 +1,6 @@
 <?xml version="1.0" encoding="UTF-8"?>
 <robot xmlns:xacro="http://ros.org/wiki/xacro">
-   <property name="M_SCALE" value="0.001"/>
-   <property name="M_PI" value="3.14159"/>
+   <xacro:property name="M_SCALE" value="0.001"/>
+   <xacro:property name="M_PI" value="3.14159"/>
    <xacro:include filename="$(find widowx_arm_description)/urdf/common_materials.xacro" />
    <!--link name="plate_top_link"/-->
@@ -197,5 +197,5 @@
       <!-- joints -->
       <joint name="${prefix}arm_base_joint" type="fixed">
-         <insert_block name="origin" />
+         <xacro:insert_block name="origin" />
          <parent link="${parent}" />
          <child link="${prefix}arm_base_link"/>
